File: pcb/sync.kicad_pcb (KiCad board)
At the start: 2 copper layers, 19.2 x 106 mm, 54 parts, among them J1 UP_Out, J2 CLK In, J3 BP_Inv_Out, J4 BP_Out, J5 Power, P1 B100K, P2 B100K, P3 B100K, P4 B100K, SW1 Button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

Commit message: Fixed button circuit, updated pcb for smaller footprints,
Parts:
- added R23: 10k, Resistor_SMD:R_0402_1005Metric, B.Cu at (52.1, 129.2)
- added R24: 10k, Resistor_SMD:R_0402_1005Metric, B.Cu at (65.4, 129.1)
- C1, C3: footprint Capacitor_SMD:C_0805_2012Metric -> Capacitor_SMD:C_0402_1005Metric; moved to B.Cu
- C10, C12, C13, C2, C4, C5, C6, C7, C9: footprint Capacitor_SMD:C_0805_2012Metric -> Capacitor_SMD:C_0402_1005Metric
- D1: footprint Package_TO_SOT_SMD:SOT-23_Handsoldering -> Package_TO_SOT_SMD:SOT-23
- D3, D4: footprint Diode_SMD:D_SOD-123 -> Diode_SMD:D_SOD-323
- R1, R3: footprint Resistor_SMD:R_0805_2012Metric -> Resistor_SMD:R_0402_1005Metric; moved to B.Cu
- R10, R11, R12, R13, R14, R15, R16, R17, R18, R19, R2, R20, R21, R22, R4, R6, R7, R8, R9: footprint Resistor_SMD:R_0805_2012Metric -> Resistor_SMD:R_0402_1005Metric
- R5: footprint Resistor_SMD:R_0805_2012Metric -> Resistor_SMD:R_0603_1608Metric
- moved R22 13.1 mm to (55.8, 131.2), turned to 0 degrees
- moved R16 6.97 mm to (63.9, 129.6)
- moved C1 5.61 mm to (59.1, 101.8), turned to -90 degrees
- moved R1 5.54 mm to (61.0, 101.8), turned to -90 degrees
- moved R3 2.63 mm to (58.6, 87.0)
- moved R14 2.17 mm to (61.2, 96.8)
- moved C3 1.77 mm to (57.2, 87.0)
- moved R12 1.58 mm to (60.6, 137.8), turned to 180 degrees
- moved R15 1.22 mm to (59.5, 100.2)
- moved R10 0.94 mm to (59.0, 137.3)
- moved R4 0.82 mm to (55.8, 129.8)
- moved R20 0.58 mm to (64.8, 91.5)
- moved D4 0.50 mm to (62.0, 74.5)
- moved C13 0.42 mm to (55.6, 91.7)
- moved D3 0.36 mm to (58.3, 74.5)
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Connections:
- J3 pad TN: (no net) -> GND
- SW1 pad 2: GND -> +5V
- SW2 pad 2: GND -> +5V
Routing:
- net +5V: track 129.5 -> 151.1 mm, vias 0 -> 1
- net D11: track 53.3 -> 36.0 mm
- net GND: track 59.0 -> 42.1 mm, vias 23 -> 21
- net Net-(R14-Pad1): track 49.7 -> 42.1 mm
- net Net-(D5-A): track 2.78 -> 10.2 mm
- net D12: track 23.2 -> 26.9 mm
- net -12V: track 57.4 -> 61.0 mm
- net Net-(R19-Pad1): track 92.4 -> 88.9 mm
- net A3: track 20.0 -> 16.6 mm, vias 1 -> 0
- net D3: track 66.4 -> 64.3 mm
- net A2: track 35.9 -> 37.8 mm
- net Net-(U2A--): track 34.9 -> 33.0 mm
- net A1: track 19.2 -> 17.4 mm, vias 1 -> 0
- net -5VA: track 12.4 -> 13.9 mm
- net A5: track 43.1 -> 41.6 mm
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